File: main.kicad_pcb (KiCad board)
At the start: 2 copper layers, 26.7 x 19.1 mm, 24 parts, among them P1 CONN_ProMini_Up, P10 CON_SHD, P2 CONN_ProMini_Down2, P3 CON_MT, P4 CON_POLOLU_DRV8834, P5 CON_ProMini_Down, P6 CONN_SRV, U1 74AHC1G04, U2 MIC2514, U3 DRV8838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

Commit message: Modified breakout PCB design
Parts:
- added REF**: MountingHole_3mm, Mounting_Holes:MountingHole_3mm, F.Cu at (99.7, 80.6)
- added REF**: MountingHole_3mm, Mounting_Holes:MountingHole_3mm, F.Cu at (69.2, 80.6)
- added REF**: MountingHole_3mm, Mounting_Holes:MountingHole_3mm, F.Cu at (69.2, 52.7)
- added REF**: MountingHole_3mm, Mounting_Holes:MountingHole_3mm, F.Cu at (99.7, 52.7)
- moved R1 2.27 mm to (74.6, 59.6)
- moved C3 0.53 mm to (80.8, 62.4)
- renumbered REF** to __P2
Routing:
- net GND: track 31.9 -> 63.2 mm
- net VCC: track 56.1 -> 59.0 mm
- net /LIGHT: track 13.1 -> 14.9 mm
- net /SHD_DRV: track 11.6 -> 13.0 mm
- net /~STEP_SLP: track 20.8 -> 21.6 mm
- net /SOL_EN: track 9.74 -> 10.6 mm
- net /MT_STOP: track 8.86 -> 9.62 mm
- net /VREG: track 14.9 -> 14.2 mm
- net /MISO: track 8.36 -> 9.05 mm
- net /SCLK: track 8.39 -> 9.07 mm
- removed copper zone on B.Cu, net GND
- removed copper zone on F.Cu, net GND
Other:
- net class power added: clearance 0.2, trace_width 0.65, via_dia 0.6, via_drill 0.4

Commit message: Modified pcb design
Parts:
- removed the REF** at (99.7, 80.6)
- removed the REF** at (69.2, 80.6)
- removed the REF** at (69.2, 52.7)
- removed the REF** at (99.7, 52.7)
- P10: footprint perfboard:Pin_Header_Straight_1x02_Pitch1.27mm -> Connectors_Molex:Molex_PicoBlade_53048-0210
- U1: footprint TO_SOT_Packages_SMD:SOT-353 -> perfboard:SOT-353
- U3: footprint perfboard:DRV8838_DSG_8 -> perfboard:DRV8838_DSG_8_ManualSolder
- moved P4 10.3 mm to (89.7, 75.3), turned to 270 degrees
- moved R1 1.25 mm to (73.3, 59.7), turned to 0 degrees
- moved U2 0.66 mm to (81.9, 64.7)
- moved P10 0.60 mm to (81.5, 72.6)
- moved C3 0.56 mm to (80.8, 61.8)
- moved P6 0.50 mm to (88.5, 72.6)
- moved REF** 0.50 mm to (88.5, 72.6)
- moved C4 0.43 mm to (83.1, 68.8)
- moved U3 0.35 mm to (80.6, 69.8)
- moved P5 0.31 mm to (91.3, 68.3)
- moved REF** 0.30 mm to (91.3, 68.3)
- moved C5 0.28 mm to (86.2, 64.3)
- moved R2 0.11 mm to (88.0, 63.6)
- moved U4 0.08 mm to (85.3, 67.8)
- turned D1 to 0 degrees
Connections:
- P1 pad 1: /SOL_DIR -> /~STEP_SLP
- P1 pad 3: /~STEP_SLP -> /SOL_DIR
Routing:
- net /SOL_DIR: track 5.03 -> 16.5 mm
- net /BL_CS: track 15.9 -> 22.3 mm, vias 4 -> 2
- net GND: track 63.2 -> 59.0 mm, vias 5 -> 4
- net /SOL_EN: track 10.6 -> 13.6 mm, vias 1 -> 0
- net /SHD_DRV: track 13.0 -> 15.5 mm
- net /MISO: track 9.05 -> 11.4 mm
- net VCC: track 59.0 -> 61.3 mm, vias 5 -> 4
- net /VMOT: track 17.3 -> 16.1 mm
- net /BL_CI: track 5.50 -> 6.73 mm
- net /~STEP_SLP: track 21.6 -> 22.8 mm
- net /BL_DO: track 4.41 -> 5.55 mm
- net /SCLK: track 9.07 -> 10.2 mm
- net Net-(P3-Pad6): track 6.35 -> 7.35 mm
- net /LIGHT: track 14.9 -> 14.1 mm
- net /PWR_SEL: track 5.75 -> 6.41 mm
Other:
- net class Default: clearance 0.2 -> 0.199
- net class power: clearance 0.2 -> 0.199
- rule trace_clearance: 0.2 -> 0.199

Commit message: Fixed motor stopper pullup
Parts:
- turned R2 to 180 degrees
Connections:
- R2 pad 1: VCC -> /MT_STOP
- R2 pad 2: Net-(P3-Pad6) -> VCC
Routing:
- net Net-(P3-Pad6): track 7.35 -> 4.92 mm
- net /MT_DIR: track 12.5 -> 14.4 mm
- net /MT_STOP: track 10.0 -> 11.8 mm, vias 0 -> 1
- net GND: track 59.0 -> 57.8 mm
