File: main.sch (KiCad schematic (older format))
At the start: 19 parts, among them P1 CONN_ProMini_Up, P10 CON_SHD, P2 CONN_ProMini_Down2, P3 CON_MT, P4 CON_POLOLU_DRV8834, P5 CON_ProMini_Down, P6 CONN_SRV, U1 74AHC1G04, U2 MIC2514, U3 DRV8838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

Commit message: Modified breakout PCB design
Parts:
- P1: footprint Connectors_Molex:Molex_PicoBlade_53398-0771 -> Connectors_Molex:Molex_PicoBlade_53261-0771
- P3: footprint Connectors_Molex:Molex_PicoBlade_53261-0671 -> Connectors_Molex:Molex_PicoBlade_53398-0771
Changed lines of the file:
@@
 F 0 "P1" H 5300 2550 50  0000 C CNN
 F 1 "CONN_ProMini_Up" V 5400 2150 50  0000 C CNN
-F 2 "Connectors_Molex:Molex_PicoBlade_53398-0771" H 5300 2150 50  0001 C CNN
+F 2 "Connectors_Molex:Molex_PicoBlade_53261-0771" H 5300 2150 50  0001 C CNN
 F 3 "" H 5300 2150 50  0000 C CNN
 	1    5300 2150
@@
 F 0 "P3" H 9100 3500 60  0000 C CNN
 F 1 "CON_MT" H 9100 3000 60  0000 C CNN
-F 2 "Connectors_Molex:Molex_PicoBlade_53261-0671" H 9100 3150 60  0001 C CNN
+F 2 "Connectors_Molex:Molex_PicoBlade_53398-0771" H 9100 3150 60  0001 C CNN
 F 3 "" H 9100 3150 60  0000 C CNN
 	1    9100 3250

Commit message: Modified pcb design
Other:
- note added: "Use receptacle here"
- note removed: "User receptacle here"
- moved on the sheet: P1
Changed lines of the file:
@@
 Text Label 8050 2600 0    60   ~ 0
 VMOT
-Text Label 5100 2250 2    60   ~ 0
+Text Label 5100 1650 2    60   ~ 0
 SCLK
 $Comp
@@
 	1    0    0    -1
 $EndComp
-Text Label 5100 2450 2    60   ~ 0
+Text Label 5100 1450 2    60   ~ 0
 MT_STOP
 Text Label 2300 4150 2    60   ~ 0
@@
 Text Label 3000 4900 2    60   ~ 0
 MISO
-Text Label 5100 2150 2    60   ~ 0
+Text Label 5100 1750 2    60   ~ 0
 BL_CS
-Text Label 5100 2350 2    60   ~ 0
+Text Label 5100 1550 2    60   ~ 0
 MISO
 Text Label 5050 4200 2    60   ~ 0
 SHD_DRV
-Text Label 3400 6150 2    60   ~ 0
+Text Label 3700 6150 2    60   ~ 0
 STEP_STOP
 $Comp
 L GND #PWR016
 U 1 1 572B29C3
-P 3400 6250
-F 0 "#PWR016" H 3400 6000 50  0001 C CNN
-F 1 "GND" H 3400 6100 50  0000 C CNN
-F 2 "" H 3400 6250 50  0000 C CNN
-F 3 "" H 3400 6250 50  0000 C CNN
-	1    3400 6250
+P 3700 6250
+F 0 "#PWR016" H 3700 6000 50  0001 C CNN
+F 1 "GND" H 3700 6100 50  0000 C CNN
+F 2 "" H 3700 6250 50  0000 C CNN
+F 3 "" H 3700 6250 50  0000 C CNN
+	1    3700 6250
 	1    0    0    -1
 $EndComp
@@
 L CONN_01X02 #P2
 U 1 1 57326719
-P 3600 6200
-F 0 "#P2" H 3600 6050 50  0001 C CNN
-F 1 "CON_STEP_STOP" V 3750 6200 50  0000 C CNN
-F 2 "~" H 3600 6200 50  0001 C CNN
-F 3 "" H 3600 6200 50  0000 C CNN
-	1    3600 6200
+P 3900 6200
+F 0 "#P2" H 3900 6050 50  0001 C CNN
+F 1 "CON_STEP_STOP" V 4050 6200 50  0000 C CNN
+F 2 "~" H 3900 6200 50  0001 C CNN
+F 3 "" H 3900 6200 50  0000 C CNN
+	1    3900 6200
 	1    0    0    1
 $EndComp
@@
 L CONN_01X07 P1
 U 1 1 573F4852
-P 5300 2150
-F 0 "P1" H 5300 2550 50  0000 C CNN
-F 1 "CONN_ProMini_Up" V 5400 2150 50  0000 C CNN
-F 2 "Connectors_Molex:Molex_PicoBlade_53261-0771" H 5300 2150 50  0001 C CNN
-F 3 "" H 5300 2150 50  0000 C CNN
-	1    5300 2150
-	1    0    0    -1
+P 5300 1750
+F 0 "P1" H 5300 2150 50  0000 C CNN
+F 1 "CONN_ProMini_Up" V 5400 1750 50  0000 C CNN
+F 2 "Connectors_Molex:Molex_PicoBlade_53261-0771" H 5300 1750 50  0001 C CNN
+F 3 "" H 5300 1750 50  0000 C CNN
+	1    5300 1750
+	1    0    0    1
 $EndComp
 $Comp
@@
 	9850 3650 8800 3650
 Text Notes 8850 4200 0    60   ~ 0
-User receptacle here
+Use receptacle here
 Wire Wire Line
 	8350 3350 8650 3350

Commit message: Fixed motor stopper pullup
Other:
- moved on the sheet: R2
