File: ibk.sch (KiCad schematic (older format))
At the start: 19 parts, among them P1 CONN_ProMini_Up, P10 CON_SHD, P2 CONN_ProMini_Down2, P3 CON_MT, P4 CON_POLOLU_DRV8834, P5 CON_ProMini_Down, P6 CONN_SRV, U1 74AHC1G04, U2 MIC2514, U3 DRV8838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

Commit message: Modified drv8835 connector
Parts:
- removed P3: CON_MT, Connectors_Molex:Molex_PicoBlade_53398-0771, symbol CON_MT
- added P?: CON_MT_STOP, Connectors_Molex:Molex_PicoBlade_53047-0210, symbol CONN_01X02
- added P?: CON_POLOLU_DRV8835, Connectors_Molex:Molex_PicoBlade_53398-0771, symbol CON_POLOLU_DRV8835
Connections:
- net labels added: CON_MT, CON_SOL
- net labels removed: CON_MT_STOP
- wire segments 76 -> 81
Other:
- note added: "Use receptacles here"
- note removed: "Use receptacle here"
- moved on the sheet: C2, R2, U1
Changed lines of the file:
@@
 LIBS:parts
 LIBS:74xgxx
-LIBS:main-cache
 EELAYER 25 0
 EELAYER END
@@
 L 74AHC1G04 U1
 U 1 1 572A6846
-P 8150 4400
-F 0 "U1" H 8345 4515 50  0000 C CNN
-F 1 "74AHC1G04" H 8450 4250 50  0000 C CNN
-F 2 "TO_SOT_Packages_SMD:SOT-353" H 8150 4400 50  0001 C CNN
-F 3 "" H 8150 4400 50  0000 C CNN
-	1    8150 4400
+P 7800 4800
+F 0 "U1" H 7995 4915 50  0000 C CNN
+F 1 "74AHC1G04" H 8100 4650 50  0000 C CNN
+F 2 "TO_SOT_Packages_SMD:SOT-353" H 7800 4800 50  0001 C CNN
+F 3 "" H 7800 4800 50  0000 C CNN
+	1    7800 4800
 	1    0    0    -1
 $EndComp
@@
 L C_Small C2
 U 1 1 572A6CE0
-P 7800 3950
-F 0 "C2" H 7650 4000 50  0000 L CNN
-F 1 "0.1uF" H 7550 3850 50  0000 L CNN
-F 2 "Capacitors_SMD:C_0402" H 7800 3950 50  0001 C CNN
-F 3 "" H 7800 3950 50  0000 C CNN
-	1    7800 3950
+P 7450 4350
+F 0 "C2" H 7300 4400 50  0000 L CNN
+F 1 "0.1uF" H 7200 4250 50  0000 L CNN
+F 2 "Capacitors_SMD:C_0402" H 7450 4350 50  0001 C CNN
+F 3 "" H 7450 4350 50  0000 C CNN
+	1    7450 4350
 	1    0    0    -1
 $EndComp
@@
 L VCC #PWR012
 U 1 1 572A6F23
-P 8100 3800
-F 0 "#PWR012" H 8100 3650 50  0001 C CNN
-F 1 "VCC" H 8100 3950 50  0000 C CNN
-F 2 "" H 8100 3800 50  0000 C CNN
-F 3 "" H 8100 3800 50  0000 C CNN
-	1    8100 3800
+P 7750 4200
+F 0 "#PWR012" H 7750 4050 50  0001 C CNN
+F 1 "VCC" H 7750 4350 50  0000 C CNN
+F 2 "" H 7750 4200 50  0000 C CNN
+F 3 "" H 7750 4200 50  0000 C CNN
+	1    7750 4200
 	1    0    0    -1
 $EndComp
@@
 L GND #PWR013
 U 1 1 572A701B
-P 7800 4050
-F 0 "#PWR013" H 7800 3800 50  0001 C CNN
-F 1 "GND" H 7800 3900 50  0000 C CNN
-F 2 "" H 7800 4050 50  0000 C CNN
-F 3 "" H 7800 4050 50  0000 C CNN
-	1    7800 4050
+P 7450 4450
+F 0 "#PWR013" H 7450 4200 50  0001 C CNN
+F 1 "GND" H 7450 4300 50  0000 C CNN
+F 2 "" H 7450 4450 50  0000 C CNN
+F 3 "" H 7450 4450 50  0000 C CNN
+	1    7450 4450
 	1    0    0    -1
 $EndComp
@@
 L GND #PWR014
 U 1 1 572A71E7
-P 8100 4600
-F 0 "#PWR014" H 8100 4350 50  0001 C CNN
-F 1 "GND" H 8100 4450 50  0000 C CNN
-F 2 "" H 8100 4600 50  0000 C CNN
-F 3 "" H 8100 4600 50  0000 C CNN
-	1    8100 4600
+P 7750 5000
+F 0 "#PWR014" H 7750 4750 50  0001 C CNN
+F 1 "GND" H 7750 4850 50  0000 C CNN
+F 2 "" H 7750 5000 50  0000 C CNN
+F 3 "" H 7750 5000 50  0000 C CNN
+	1    7750 5000
 	1    0    0    -1
 $EndComp
@@
 L R R2
 U 1 1 572A7BCC
-P 9900 3300
-F 0 "R2" V 9800 3300 50  0000 C CNN
-F 1 "10K" V 9900 3300 50  0000 C CNN
-F 2 "Resistors_SMD:R_0402" V 9830 3300 50  0001 C CNN
-F 3 "" H 9900 3300 50  0000 C CNN
-	1    9900 3300
-	1    0    0    -1
+P 8050 4250
+F 0 "R2" V 7950 4250 50  0000 C CNN
+F 1 "10K" V 8050 4250 50  0000 C CNN
+F 2 "Resistors_SMD:R_0402" V 7980 4250 50  0001 C CNN
+F 3 "" H 8050 4250 50  0000 C CNN
+	1    8050 4250
+	0    1    1    0
 $EndComp
 $Comp
 L VCC #PWR015
 U 1 1 572A7C9B
-P 9900 3150
-F 0 "#PWR015" H 9900 3000 50  0001 C CNN
-F 1 "VCC" H 9900 3300 50  0000 C CNN
-F 2 "" H 9900 3150 50  0000 C CNN
-F 3 "" H 9900 3150 50  0000 C CNN
-	1    9900 3150
+P 8100 3050
+F 0 "#PWR015" H 8100 2900 50  0001 C CNN
+F 1 "VCC" H 8100 3200 50  0000 C CNN
+F 2 "" H 8100 3050 50  0000 C CNN
+F 3 "" H 8100 3050 50  0000 C CNN
+	1    8100 3050
 	1    0    0    -1
 $EndComp
@@
 L GND #PWR020
 U 1 1 572D09A7
-P 9550 3350
-F 0 "#PWR020" H 9550 3100 50  0001 C CNN
-F 1 "GND" H 9550 3200 50  0000 C CNN
-F 2 "" H 9550 3350 50  0000 C CNN
-F 3 "" H 9550 3350 50  0000 C CNN
-	1    9550 3350
+P 8100 3250
+F 0 "#PWR020" H 8100 3000 50  0001 C CNN
+F 1 "GND" H 8100 3100 50  0000 C CNN
+F 2 "" H 8100 3250 50  0000 C CNN
+F 3 "" H 8100 3250 50  0000 C CNN
+	1    8100 3250
 	1    0    0    -1
 $EndComp
@@
 	1    0    0    -1
 $EndComp
-Text Label 8650 3350 2    60   ~ 0
+Text Label 8650 3650 2    60   ~ 0
 MT_STOP
 $Comp
@@
 	1    0    0    -1
 $EndComp
-Text Label 7200 4400 2    60   ~ 0
+Text Label 6850 4800 2    60   ~ 0
 MT_DIR
 $Comp
@@
 $EndComp
 $Comp
-L CONN_01X02 #P3
+L CONN_01X02 P?
 U 1 1 573F5023
-P 9100 3850
-F 0 "#P3" H 9100 3700 50  0001 C CNN
-F 1 "CON_MT_STOP" H 9100 4000 50  0000 C CNN
-F 2 "perfboard:Pin_Header_Straight_1x02_Pitch1.27mm" H 9100 3850 50  0001 C CNN
-F 3 "" H 9100 3850 50  0000 C CNN
-	1    9100 3850
+P 8800 4750
+F 0 "P?" H 8800 4600 50  0000 C CNN
+F 1 "CON_MT_STOP" H 8800 4900 50  0000 C CNN
+F 2 "Connectors_Molex:Molex_PicoBlade_53047-0210" H 8800 4750 50  0001 C CNN
+F 3 "" H 8800 4750 50  0000 C CNN
+	1    8800 4750
 	1    0    0    1
 $EndComp
@@
 	6850 2550 6950 2550
 Wire Wire Line
-	7200 4400 7700 4400
-Wire Wire Line
-	8100 3800 8100 4200
+	6850 4800 7350 4800
+Wire Wire Line
+	7750 4200 7750 4600
 Wire Wire Line
 	2300 4150 3450 4150
@@
 	3500 3800 3750 3800
 Connection ~ 8750 2450
-Connection ~ 8100 3850
-Wire Wire Line
-	7800 3850 8100 3850
+Connection ~ 7750 4250
+Wire Wire Line
+	7450 4250 7900 4250
 Wire Wire Line
 	9000 1800 9350 1800
@@
 Wire Wire Line
 	9000 1900 9250 1900
-Connection ~ 9900 3450
 Wire Wire Line
 	8050 2600 8300 2600
@@
 Wire Wire Line
 	6850 1850 6850 2550
-Connection ~ 9900 3150
 Wire Wire Line
 	6350 1200 6350 1950
@@
 Text Notes 3200 5800 0    60   ~ 0
 Make this receptacle
-$Comp
-L CON_MT P3
-U 1 1 573FEAA2
-P 9100 3250
-F 0 "P3" H 9100 3500 60  0000 C CNN
-F 1 "CON_MT" H 9100 3000 60  0000 C CNN
-F 2 "Connectors_Molex:Molex_PicoBlade_53398-0771" H 9100 3150 60  0001 C CNN
-F 3 "" H 9100 3150 60  0000 C CNN
-	1    9100 3250
-	1    0    0    -1
-$EndComp
 Wire Wire Line
 	8050 2750 8300 2750
-Wire Wire Line
-	8300 2600 8300 3150
-Wire Wire Line
-	8300 3150 8650 3150
 Connection ~ 8300 2750
-Wire Wire Line
-	8600 4400 9900 4400
-Wire Wire Line
-	9900 4400 9900 3450
-Wire Wire Line
-	9900 3150 9550 3150
-Wire Wire Line
-	9550 3250 9700 3250
-Wire Wire Line
-	9700 3250 9700 3450
-Wire Wire Line
-	9700 3450 9900 3450
-Wire Wire Line
-	8650 3250 7400 3250
-Wire Wire Line
-	7400 3250 7400 4400
-Connection ~ 7400 4400
-Wire Wire Line
-	8350 3350 8350 3800
-Wire Wire Line
-	8350 3800 8900 3800
-Wire Wire Line
-	8900 3900 8700 3900
-Wire Wire Line
-	8700 3900 8700 4400
-Connection ~ 8700 4400
-Wire Notes Line
-	8800 3650 8800 4300
-Wire Notes Line
-	8800 4300 9850 4300
-Wire Notes Line
-	9850 4300 9850 3650
-Wire Notes Line
-	9850 3650 8800 3650
-Text Notes 8850 4200 0    60   ~ 0
-Use receptacle here
-Wire Wire Line
-	8350 3350 8650 3350
+Connection ~ 7050 4800
+Text Notes 9750 3650 0    60   ~ 0
+Use receptacles here
 $Comp
 L CONN_01X05 P2
@@
 	-1   0    0    1
 $EndComp
+Wire Wire Line
+	8300 2600 8300 3050
+Wire Wire Line
+	8300 3050 8650 3050
+Text Label 8650 3350 2    60   ~ 0
+SOL_DIR
+Text Label 8650 3450 2    60   ~ 0
+SOL_EN
+$Comp
+L CONN_01X02 #P?
+U 1 1 576CC17A
+P 10000 3400
+F 0 "#P?" H 10000 3250 50  0001 C CNN
+F 1 "CON_SOL" H 10250 3400 50  0000 C CNN
+F 2 "perfboard:Pin_Header_Straight_1x02_Pitch1.27mm" H 10000 3400 50  0001 C CNN
+F 3 "" H 10000 3400 50  0000 C CNN
+	1    10000 3400
+	1    0    0    1
+$EndComp
+$Comp
+L CONN_01X02 #P?
+U 1 1 576CC1D5
+P 10000 3100
+F 0 "#P?" H 10000 2950 50  0001 C CNN
+F 1 "CON_MT" H 10200 3100 50  0000 C CNN
+F 2 "perfboard:Pin_Header_Straight_1x02_Pitch1.27mm" H 10000 3100 50  0001 C CNN
+F 3 "" H 10000 3100 50  0000 C CNN
+	1    10000 3100
+	1    0    0    1
+$EndComp
+$Comp
+L CON_POLOLU_DRV8835 P?
+U 1 1 576CD25C
+P 9100 3250
+F 0 "P?" H 9100 3600 60  0000 C CNN
+F 1 "CON_POLOLU_DRV8835" H 9100 2700 60  0000 C CNN
+F 2 "Connectors_Molex:Molex_PicoBlade_53398-0771" H 9000 3100 60  0001 C CNN
+F 3 "" H 9000 3100 60  0000 C CNN
+	1    9100 3250
+	1    0    0    -1
+$EndComp
+Wire Wire Line
+	7050 4800 7050 3550
+Wire Wire Line
+	7050 3550 8650 3550
+Wire Wire Line
+	8100 3050 8100 3150
+Wire Wire Line
+	8100 3150 8650 3150
+Wire Wire Line
+	8650 3250 8100 3250
+Wire Wire Line
+	9550 3050 9800 3050
+Wire Wire Line
+	9550 3150 9800 3150
+Wire Wire Line
+	9550 3250 9700 3250
+Wire Wire Line
+	9700 3250 9700 3350
+Wire Wire Line
+	9700 3350 9800 3350
+Wire Wire Line
+	9550 3350 9600 3350
+Wire Wire Line
+	9600 3350 9600 3450
+Wire Wire Line
+	9600 3450 9800 3450
+Wire Notes Line
+	9650 2950 9650 3700
+Wire Notes Line
+	9650 3700 10850 3700
+Wire Notes Line
+	10850 3700 10850 2950
+Wire Notes Line
+	10850 2950 9650 2950
+Wire Wire Line
+	8250 4800 8600 4800
+Wire Wire Line
+	8650 3650 8350 3650
+Wire Wire Line
+	8350 3650 8350 4700
+Wire Wire Line
+	8350 4700 8600 4700
+Wire Wire Line
+	8200 4250 8350 4250
+Connection ~ 8350 4250
 $EndSCHEMATC

Commit message: Fixed schematics
Parts:
- removed R2: 10K, Resistors_SMD:R_0402, symbol R
- removed unit 1 of U4
- P?: symbol CON_POLOLU_DRV8835 -> CON_POLOLU_DRV8835-RESCUE-ibk
Connections:
- net labels added: MT_EN, ~SHD_SLP
- net labels removed: BL_DO, MISO, MT_STOP
- wire segments 81 -> 72
Other:
- note added: "Inverter abandoned.\nUse MCU output pin for ~MT_DIR,\nso that we can make it input and set\nMT_EN as output to force stop motor."
- moved on the sheet: P?
